Commit message: modifying launch file , editing sensors features

File: waiteronix/urdf/waiteronix.xacro (robot description, xacro)
@@ -1,6 +1,9 @@
-<robot name="waiteronix">
+<robot name="waiteronix" xmlns:xacro="http://www.ros.org/wiki/xacro">
   <!-- This URDF was automatically created by SolidWorks to URDF Exporter! Originally created by Stephen Brawner (brawner@gmail.com)
      Commit Version: 1.6.0-4-g7f85cfe  Build Version: 1.6.7995.38578
      For more information, please see http://wiki.ros.org/sw_urdf_exporter -->
+  <xacro:include filename="$(find waiteronix)/urdf/rrbot.gazebo"/>
+  <link name="robot_footprint">
+  </link>
   <link
     name="base_link">
@@ -83,4 +86,8 @@
     </collision>
   </link>
+    <joint name="dummy_joint" type="fixed">
+    <parent link="robot_footprint"/>
+    <child link="base_link"/>
+   </joint>
   <joint
     name="Body_Joint"
@@ -579,68 +586,3 @@
       xyz="0 1 0" />
   </joint>
-  <gazebo reference="Camera">
-  <sensor name="Camera_camera" type="depth">
-    <update_rate>20</update_rate>
-    <camera>
-      <horizontal_fov>1.047198</horizontal_fov>
-      <image>
-        <width>640</width>
-        <height>480</height>
-        <format>R8G8B8</format>
-      </image>
-      <clip>
-        <near>0.05</near>
-        <far>3</far>
-      </clip>
-    </camera>
-    <plugin name="Camera_controller" filename="libgazebo_ros_openni_kinect.so">
-      <baseline>0.2</baseline>
-      <alwaysOn>true</alwaysOn>
-      <updateRate>1.0</updateRate>
-      <cameraName>Camera_ir</cameraName>
-      <imageTopicName>/Camera/color/image_raw</imageTopicName>
-      <cameraInfoTopicName>/Camera/color/camera_info</cameraInfoTopicName>
-      <depthImageTopicName>/Camera/depth/image_raw</depthImageTopicName>
-      <depthImageInfoTopicName>/Camera/depth/camera_info</depthImageInfoTopicName>
-      <pointCloudTopicName>/Camera/depth/points</pointCloudTopicName>
-      <frameName>camera_link</frameName>
-      <pointCloudCutoff>0.5</pointCloudCutoff>
-      <pointCloudCutoffMax>3.0</pointCloudCutoffMax>
-      <distortionK1>0.00000001</distortionK1>
-      <distortionK2>0.00000001</distortionK2>
-      <distortionK3>0.00000001</distortionK3>
-      <distortionT1>0.00000001</distortionT1>
-      <distortionT2>0.00000001</distortionT2>
-      <CxPrime>0</CxPrime>
-      <Cx>0</Cx>
-      <Cy>0</Cy>
-      <focalLength>0</focalLength>
-      <hackBaseline>0</hackBaseline>
-    </plugin>
-  </sensor>
-   </gazebo>
-    <gazebo reference="Lidar">
-        <sensor type="ray" name="laser" >
-            <pose> 0 0 0 0 0 0 </pose>
-            <visualize>true</visualize>
-            <update_rate>10</update_rate>
-            <ray>
-                <scan>
-                    <horizontal>
-                        <samples>360</samples>
-                        <min_angle>-3.14</min_angle>
-                        <max_angle>3.14</max_angle>
-                    </horizontal>
-                </scan>
-                <range>
-                    <min>0.3</min>
-                    <max>12</max>
-                </range>
-            </ray>
-            <plugin name="Lidar_controller" filename="libgazebo_ros_ray_sensor.so">
-                 <topicName>/scan</topicName>
-                <frame_name>Lidar</frame_name>
-            </plugin>
-        </sensor>
-    </gazebo>
 </robot>
